Commit message: add the visual and mass in the model

File: catkin_ws/src/ligong_description/urdf/ligong.xacro (robot description, xacro)
@@ -8,3 +8,20 @@
 		<child link = "link" />
 	</joint>
+<!--Base link-->
+<!--add the visual model-->
+<visual>
+	<origin xyz = "0 0 0.5" rpy= "0 0 0 "/>
+	<geometry>
+		<box size = "0.2 0.2 1" />
+	</geometry>
+</visual>
+<!--the mass-->
+<inertial>
+	<origin xyz ="0 0 0.5" rpy="0 0 0"/>
+	<mass value ="1" />
+	<inertia
+		ixx = "1.0" ixy = "0.0" ixz = "0.0"
+		iyy = "1.0" iyz = "0.0"
+		izz = "1.0"/>
+</inertial>
 </robot>

Commit message: add the collision of our urdf

File: catkin_ws/src/ligong_description/urdf/ligong.xacro (robot description, xacro)
@@ -10,4 +10,7 @@
 <!--Base link-->
 <!--add the visual model-->
+<collision>
+	<origin xyz = "0 0 0.5" rpy= "0 0 0 "/>
+</collision>
 <visual>
 	<origin xyz = "0 0 0.5" rpy= "0 0 0 "/>
@@ -21,7 +24,7 @@
 	<mass value ="1" />
 	<inertia
-		ixx = "1.0" ixy = "0.0" ixz = "0.0"
+		ixx = "1.0" ixy = "0.0"  ixz="0.0"
 		iyy = "1.0" iyz = "0.0"
-		izz = "1.0"/>
+		izz = "1.0" />
 </inertial>
 </robot>

Commit message: add the collision

File: catkin_ws/src/ligong_description/urdf/ligong.xacro (robot description, xacro)
@@ -9,7 +9,9 @@
 	</joint>
 <!--Base link-->
-<!--add the visual model-->
+<!--add the visual mode-->
 <collision>
-	<origin xyz = "0 0 0.5" rpy= "0 0 0 "/>
+	<geometry>
+		<box size = "0.2 0.0 1"/>
+	</geometry>
 </collision>
 <visual>
